File: Prototype1/CAD Files/B1.kicad_pcb (KiCad board)
At the start: 2 copper layers, 18 parts, among them U1 ArduinoProMini, U2 PE4259

Commit message: Added Stuff
Parts:
- moved TP2 79.9 mm to (125.2, 67.8)
- moved TP3 64.7 mm to (125.0, 95.8)
- moved C1 60.7 mm to (140.5, 90.4)
- moved TP4 54.8 mm to (125.0, 108.0)
- moved AE2 40.6 mm to (125.9, 80.8)
- moved TP7 39.9 mm to (136.4, 138.9)
- moved TP6 39.9 mm to (152.4, 139.2)
- moved U1 34.5 mm to (146.2, 109.4), turned to 180 degrees
- moved TP5 33.9 mm to (152.7, 132.1)
- moved R1 32.3 mm to (140.6, 88.2)
- moved R2 26.4 mm to (138.0, 89.3), turned to 90 degrees
- moved U2 24.1 mm to (132.1, 87.3), turned to 180 degrees
- moved L1 18.5 mm to (135.3, 88.2), turned to 180 degrees
- moved TP9 18.2 mm to (143.8, 139.2)
- moved RX1-1 15.5 mm to (137.2, 115.6), turned to 270 degrees
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Routing:
- net Net-(TP5-Pad1): track 0.00 -> 21.6 mm
- net /RF_Switched: track 0.00 -> 12.9 mm
- net Net-(RX1-1-Pad8): track 0.00 -> 12.1 mm
- net /RF_Right: track 0.00 -> 7.96 mm
- net /RF_Left: track 0.00 -> 7.80 mm
- net /Control/RF_CLK: track 0.00 -> 7.15 mm
- net Net-(L1-Pad1): track 0.00 -> 3.26 mm
- net GND: track 0.00 -> 2.50 mm
- net Net-(L1-Pad2): track 0.00 -> 1.19 mm
- net +3V3: track 0.00 -> 0.09 mm, vias 0 -> 1
- added copper zone on B.Cu, net +3V3
- added copper zone on F.Cu, net GND
Other:
- board outline added: 43.2 x 85.1 mm
