File: Prototype1/CAD Files/_autosave-B1.kicad_pcb (KiCad board)
At the start: 2 copper layers, 43.2 x 85.1 mm, 18 parts, among them U1 ArduinoProMini, U2 PE4259

Commit message: Added Stuff
Changed lines of the file:
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@@
     (visible_elements 7FFFFFFF)
     (pcbplotparams
-      (layerselection 0x00030_80000001)
+      (layerselection 0x01000_80000001)
       (usegerberextensions false)
       (excludeedgelayer true)
@@
       (padsonsilk false)
       (subtractmaskfromsilk false)
-      (outputformat 4)
+      (outputformat 1)
       (mirror false)
       (drillshape 0)
@@
       (effects (font (size 1 1) (thickness 0.15)))
     )
+    (fp_line (start -1.016 0.254) (end -1.27 0.254) (layer F.SilkS) (width 0.15))
+    (fp_line (start -1.016 -0.254) (end -1.016 0.254) (layer F.SilkS) (width 0.15))
+    (fp_line (start -1.27 -0.254) (end -1.016 -0.254) (layer F.SilkS) (width 0.15))
+    (fp_line (start 1.27 0.889) (end 1.27 -0.889) (layer F.SilkS) (width 0.15))
+    (fp_line (start -1.27 0.889) (end 1.27 0.889) (layer F.SilkS) (width 0.15))
+    (fp_line (start -1.27 -0.889) (end -1.27 0.889) (layer F.SilkS) (width 0.15))
+    (fp_line (start 1.27 -0.889) (end -1.27 -0.889) (layer F.SilkS) (width 0.15))
     (pad 1 smd rect (at -0.65 0.9 180) (size 0.47 1) (layers F.Cu F.Paste F.Mask)
       (net 1 /RF_Right))
